File: circuit_board/smart_clock_button.kicad_pcb (KiCad board)
At the start: 2 copper layers, 25.4 x 11.5 mm, 5 parts, among them J1 Conn_01x01_Socket, J2 Conn_01x01_Socket, SW1 SW_Push

Commit message: Updated circuit board
Other:
- board text added: "Rev A"
- board text added: "Smart Clock"
Changed lines of the file:
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@@
 		(property "Reference" "J1"
 			(at 0 -1.648 0)
-			(layer "F.SilkS")
-			(effects
-				(font
-					(size 1 1)
-					(thickness 0.15)
-				)
+			(layer "B.SilkS")
+			(effects
+				(font
+					(size 1 1)
+					(thickness 0.15)
+				)
+				(justify mirror)
 			)
 		)
@@
 		(property "Reference" "J2"
 			(at 0 -1.648 0)
-			(layer "F.SilkS")
-			(effects
-				(font
-					(size 1 1)
-					(thickness 0.15)
-				)
+			(layer "B.SilkS")
+			(effects
+				(font
+					(size 1 1)
+					(thickness 0.15)
+				)
+				(justify mirror)
 			)
 		)
@@
 		(layer "Edge.Cuts")
 	)
+	(gr_text "Smart Clock"
+		(at 151 84.4 0)
+		(layer "F.SilkS")
+		(effects
+			(font
+				(size 1.5 1.5)
+				(thickness 0.3)
+				(bold yes)
+			)
+			(justify bottom)
+		)
+	)
+	(gr_text "Rev A"
+		(at 145 85.4 0)
+		(layer "F.SilkS")
+		(effects
+			(font
+				(size 0.5 0.5)
+				(thickness 0.125)
+			)
+			(justify left bottom)
+		)
+	)
 	(segment
